Commit message: msgs added

File: src/smart_car/urdf/smartcar.urdf (robot description, URDF)
Before this commit: robot smartcar, 6 links, 5 joints
Links:
- removed link rear_left_wheel
- removed link rear_right_wheel
- added link back_left_wheel, mass 0.2; visual cylinder length=0.025 radius=0.032
- added link back_right_wheel, mass 0.2; visual cylinder length=0.025 radius=0.032
- added link imu_link
- added link sllidar_base_link
- link chassis_link: mass None -> 1.0
- link front_left_wheel: mass None -> 0.2
- link front_right_wheel: mass None -> 0.2
Joints:
- removed joint rear_left_wheel_joint
- removed joint rear_right_wheel_joint
- added joint back_left_wheel_joint: type continuous, parent base_link, child back_left_wheel, origin xyz=0.11000000000000001 0.1285 0.032 rpy=0 1.5707963267948966 0
- added joint back_right_wheel_joint: type continuous, parent base_link, child back_right_wheel, origin xyz=-0.11000000000000001 0.1285 0.032 rpy=0 1.5707963267948966 0

File: src/smart_car/urdf/smartcar.urdf.xacro (robot description, xacro)
@@ -1,4 +1,4 @@
-<?xml version="1.0"?>
 <robot xmlns:xacro="http://www.ros.org/wiki/xacro" name="smartcar">
+  <!--Xacro properties and macros-->
   <xacro:property name="wheel_diameter" value="0.064" />
   <xacro:property name="wheel_width" value="0.025" />
@@ -7,4 +7,9 @@
   <xacro:macro name="wheel" params="prefix parent x y z">
     <link name="${prefix}_wheel">
+      <inertial>
+        <mass value="0.2"/>
+        <inertia ixx="0.0001" ixy="0.0" ixz="0.0" iyy="0.0001" iyz="0.0" izz="0.0002"/>
+        <origin xyz="0 0 0"/>
+      </inertial>
       <visual>
         <geometry>
@@ -16,16 +21,20 @@
       <parent link="${parent}" />
       <child link="${prefix}_wheel"/>
-       <origin xyz="${x} ${y} ${z}" rpy="0 ${pi/2} 0"/>
+      <origin xyz="${x} ${y} ${z}" rpy="0 ${pi/2} 0"/>
     </joint>
   </xacro:macro>
+  <!--Body-->
   <link name="base_link">
     <visual>
       <geometry>
-        <!-- <box size="${wheelbase_width} ${wheelbase_length}  0.01"/>
-        <origin xyz="0 0 ${wheel_diameter / 2}"/> -->
       </geometry>
     </visual>
   </link>
-    <link name="chassis_link">
+  <link name="chassis_link">
+    <inertial>
+      <mass value="1.0"/>
+      <inertia ixx="0.01" ixy="0.0" ixz="0.0" iyy="0.01" iyz="0.0" izz="0.02"/>
+      <origin xyz="0 0 0"/>
+    </inertial>
     <visual>
       <geometry>
@@ -34,12 +43,48 @@
     </visual>
   </link>
-      <joint name="chassis_joint" type="fixed">
-      <parent link="base_link" />
-      <child link="chassis_link"/>
-      <origin xyz="0 0 ${wheel_diameter / 2}"/>
+  <joint name="chassis_joint" type="fixed">
+    <parent link="base_link" />
+    <child link="chassis_link"/>
+    <origin xyz="0 0 ${wheel_diameter / 2}"/>
   </joint>
-  <xacro:wheel prefix="front_left"  parent="base_link" x="${wheelbase_width / 2 + wheel_width}" y="-${wheelbase_length / 2}" z="${wheel_diameter / 2}"/>
+  <xacro:wheel prefix="front_left" parent="base_link" x="${wheelbase_width / 2 + wheel_width}" y="-${wheelbase_length / 2}" z="${wheel_diameter / 2}"/>
   <xacro:wheel prefix="front_right" parent="base_link" x="-${wheelbase_width / 2 + wheel_width}" y="-${wheelbase_length / 2}" z="${wheel_diameter / 2}"/>
-  <xacro:wheel prefix="back_left"   parent="base_link" x="${wheelbase_width / 2 + wheel_width}" y="${wheelbase_length / 2}" z="${wheel_diameter / 2}"/>
-  <xacro:wheel prefix="back_right"  parent="base_link" x="-${wheelbase_width / 2 + wheel_width}" y="${wheelbase_length / 2}" z="${wheel_diameter / 2}"/>
+  <xacro:wheel prefix="back_left" parent="base_link" x="${wheelbase_width / 2 + wheel_width}" y="${wheelbase_length / 2}" z="${wheel_diameter / 2}"/>
+  <xacro:wheel prefix="back_right" parent="base_link" x="-${wheelbase_width / 2 + wheel_width}" y="${wheelbase_length / 2}" z="${wheel_diameter / 2}"/>
+  <!--Sensors-->
+  <!--IMU-->
+  <link name="imu_link">
+    <!--TODO: add visual-->
+  </link>
+  <!-- <joint name="imu_joint" type="fixed">
+    <parent link="base_link" />
+    <child link="imu_link"/>
+    <origin xyz="0 0 ${wheel_diameter / 2}"/>
+  </joint>
+  <gazebo reference="imu_link">
+    <sensor type="imu" name="imu_sensor">
+      <plugin name="gazebo_ros_imu_sensor" filename="libgazebo_ros_imu_sensor.so">
+      <topicName>imu_data</topicName>
+      <frame_name>imu_link</frame_name>
+      </plugin>
+    </sensor>
+  </gazebo> -->
+  <!--LiDAR-->
+  <link name="sllidar_base_link">
+    <!--TODO: add visual-->
+  </link>
+  <!-- <joint name="lidar_joint" type="fixed">
+    <parent link="base_link" />
+    <child link="sllidar_base_link"/>
+    <origin xyz="0 0 ${wheel_diameter / 2}"/>
+  </joint>
+  <gazebo reference="sllidar_base_link">
+    <sensor type="lidar" name="imu_sensor">
+      <plugin name="gazebo_ros_imu_sensor" filename="libgazebo_ros_ray_sensor.so">
+      <output_type>sensor_msgs/Laserscan</output_type>
+      <topicName>scan</topicName>
+      <frame_name>sllidar_base_link</frame_name>
+      </plugin>
+    </sensor>
+  </gazebo> -->
 </robot>

Commit message: werkt niet

File: src/smart_car/urdf/smartcar.urdf (robot description, URDF)
Before this commit: robot smartcar, 8 links, 5 joints
Links:
- removed link imu_link
- removed link sllidar_base_link

File: src/smart_car/urdf/smartcar.urdf.xacro (robot description, xacro)
@@ -1,2 +1,3 @@
+<?xml version="1.0"?>
 <robot xmlns:xacro="http://www.ros.org/wiki/xacro" name="smartcar">
   <!--Xacro properties and macros-->
@@ -26,8 +27,4 @@
   <!--Body-->
   <link name="base_link">
-    <visual>
-      <geometry>
-      </geometry>
-    </visual>
   </link>
   <link name="chassis_link">
@@ -54,25 +51,28 @@
   <!--Sensors-->
   <!--IMU-->
-  <link name="imu_link">
-    <!--TODO: add visual-->
+  <!-- <link name="imu_link">
+    <sensor name="imu_sensor" type="imu">
+      <always_on>true</always_on> -->
+      <!-- Publish at 30 hz -->
+      <!-- <update_rate>30</update_rate>
+      <plugin name="gazebo_ros_imu_sensor" filename="libgazebo_ros_imu_sensor.so">
+        <ros> -->
+          <!-- Will publish to /imu/data -->
+          <!-- <namespace>/imu</namespace>
+          <remapping>~/out:=data</remapping>
+        </ros>
+      </plugin>
+    </sensor>
   </link>
-  <!-- <joint name="imu_joint" type="fixed">
+  <joint name="imu_joint" type="fixed">
     <parent link="base_link" />
     <child link="imu_link"/>
     <origin xyz="0 0 ${wheel_diameter / 2}"/>
-  </joint>
-  <gazebo reference="imu_link">
-    <sensor type="imu" name="imu_sensor">
-      <plugin name="gazebo_ros_imu_sensor" filename="libgazebo_ros_imu_sensor.so">
-      <topicName>imu_data</topicName>
-      <frame_name>imu_link</frame_name>
-      </plugin>
-    </sensor>
-  </gazebo> -->
-  <!--LiDAR-->
-  <link name="sllidar_base_link">
-    <!--TODO: add visual-->
-  </link>
-  <!-- <joint name="lidar_joint" type="fixed">
+  </joint> -->
+  <!-- LiDAR -->
+  <!-- <link name="sllidar_base_link"> -->
+    <!-- TODO: add visual for LiDAR -->
+  <!-- </link>
+  <joint name="lidar_joint" type="fixed">
     <parent link="base_link" />
     <child link="sllidar_base_link"/>
@@ -80,9 +80,9 @@
   </joint>
   <gazebo reference="sllidar_base_link">
-    <sensor type="lidar" name="imu_sensor">
-      <plugin name="gazebo_ros_imu_sensor" filename="libgazebo_ros_ray_sensor.so">
-      <output_type>sensor_msgs/Laserscan</output_type>
-      <topicName>scan</topicName>
-      <frame_name>sllidar_base_link</frame_name>
+    <sensor type="ray" name="lidar_sensor">
+      <update_rate>30.0</update_rate>
+      <plugin name="gazebo_ros_ray_sensor" filename="libgazebo_ros_ray_sensor.so">
+        <topic>/scan</topic>
+        <frameName>sllidar_base_link</frameName>
       </plugin>
     </sensor>

Commit message: niks werkt

File: src/smart_car/urdf/smartcar.urdf (robot description, URDF)
Before this commit: robot smartcar, 6 links, 5 joints
Links:
- added link imu_link, mass 0.05; visual box size=0.05 0.05 0.05
- added link sllidar_base_link, mass 0.05; visual cylinder length=0.1 radius=0.03
Joints:
- added joint imu_joint: type fixed, parent base_link, child imu_link, origin xyz=0 0 0.082
- added joint lidar_joint: type fixed, parent base_link, child sllidar_base_link, origin xyz=0 0 0.132

File: src/smart_car/urdf/smartcar.urdf.xacro (robot description, xacro)
@@ -51,31 +51,50 @@
   <!--Sensors-->
   <!--IMU-->
-  <!-- <link name="imu_link">
-    <sensor name="imu_sensor" type="imu">
-      <always_on>true</always_on> -->
-      <!-- Publish at 30 hz -->
-      <!-- <update_rate>30</update_rate>
-      <plugin name="gazebo_ros_imu_sensor" filename="libgazebo_ros_imu_sensor.so">
-        <ros> -->
-          <!-- Will publish to /imu/data -->
-          <!-- <namespace>/imu</namespace>
-          <remapping>~/out:=data</remapping>
-        </ros>
-      </plugin>
-    </sensor>
+  <link name="imu_link">
+    <inertial>
+      <mass value="0.05"/>
+      <origin xyz="0 0 0"/>
+    </inertial>
+    <visual>
+      <geometry>
+        <box size="0.05 0.05 0.05"/>
+      </geometry>
+      <material name="green"/>
+    </visual>
   </link>
   <joint name="imu_joint" type="fixed">
     <parent link="base_link" />
     <child link="imu_link"/>
-    <origin xyz="0 0 ${wheel_diameter / 2}"/>
-  </joint> -->
+    <origin xyz="0 0 ${wheel_diameter / 2 + 0.05}"/>
+  </joint>
+  <gazebo reference="imu_link">
+    <sensor type="imu" name="imu_sensor">
+      <always_on>true</always_on>
+      <update_rate>30.0</update_rate>
+      <plugin name="gazebo_ros_imu" filename="libgazebo_ros_imu.so">
+        <ros>
+          <namespace>/imu</namespace>
+          <remapping>~/out:=/imu/data</remapping>
+        </ros>
+      </plugin>
+    </sensor>
+  </gazebo>
   <!-- LiDAR -->
-  <!-- <link name="sllidar_base_link"> -->
-    <!-- TODO: add visual for LiDAR -->
-  <!-- </link>
+  <link name="sllidar_base_link">
+    <inertial>
+      <mass value="0.05"/>
+      <origin xyz="0 0 0"/>
+    </inertial>
+    <visual>
+      <geometry>
+        <cylinder radius="0.03" length="0.1"/>
+      </geometry>
+      <material name="red"/>
+    </visual>
+  </link>
   <joint name="lidar_joint" type="fixed">
     <parent link="base_link" />
     <child link="sllidar_base_link"/>
-    <origin xyz="0 0 ${wheel_diameter / 2}"/>
+    <origin xyz="0 0 ${wheel_diameter / 2 + 0.1}"/>
   </joint>
   <gazebo reference="sllidar_base_link">
@@ -87,4 +106,4 @@
       </plugin>
     </sensor>
-  </gazebo> -->
+  </gazebo>
 </robot>

Commit message: sensoren bestaan

File: src/smart_car/urdf/smartcar.urdf (robot description, URDF)
Before this commit: robot smartcar, 8 links, 7 joints
Links:
- link imu_link: geometry collision box size=0.1 0.1 0.1; visual box size=0.05 0.05 0.05
- link sllidar_base_link: geometry collision cylinder length=0.1 radius=0.03; visual cylinder length=0.1 radius=0.03
Joints:
- joint lidar_joint: origin xyz=0 0 0.132 -> xyz=0 0.0985 0.132

File: src/smart_car/urdf/smartcar.urdf.xacro (robot description, xacro)
@@ -6,4 +6,5 @@
   <xacro:property name="wheelbase_length" value="0.257" />
   <xacro:property name="wheelbase_width" value="0.17" />
+  <xacro:property name="LiDAR_radius" value="0.03" />
   <xacro:macro name="wheel" params="prefix parent x y z">
     <link name="${prefix}_wheel">
@@ -52,14 +53,20 @@
   <!--IMU-->
   <link name="imu_link">
-    <inertial>
-      <mass value="0.05"/>
-      <origin xyz="0 0 0"/>
-    </inertial>
     <visual>
       <geometry>
         <box size="0.05 0.05 0.05"/>
       </geometry>
-      <material name="green"/>
     </visual>
+    <collision>
+      <origin xyz="0 0 0" rpy="0 0 0"/>
+      <geometry>
+          <box size="0.1 0.1 0.1"/>
+      </geometry>
+    </collision>
+    <inertial>
+      <mass value="0.05"/>
+      <inertia ixx="0.01" ixy="0.0" ixz="0.0" iyy="0.01" iyz="0.0" izz="0.02"/>
+      <origin xyz="0 0 0"/>
+    </inertial>
   </link>
   <joint name="imu_joint" type="fixed">
@@ -82,19 +89,25 @@
   <!-- LiDAR -->
   <link name="sllidar_base_link">
+    <visual>
+      <geometry>
+        <cylinder radius="${LiDAR_radius}" length="0.1"/>
+      </geometry>
+    </visual>
+    <collision>
+      <origin xyz="0 0 0" rpy="0 0 0"/>
+      <geometry>
+        <cylinder radius="${LiDAR_radius}" length="0.1"/>
+      </geometry>
+    </collision>
     <inertial>
       <mass value="0.05"/>
+      <inertia ixx="0.01" ixy="0.0" ixz="0.0" iyy="0.01" iyz="0.0" izz="0.02"/>
       <origin xyz="0 0 0"/>
     </inertial>
-    <visual>
-      <geometry>
-        <cylinder radius="0.03" length="0.1"/>
-      </geometry>
-      <material name="red"/>
-    </visual>
   </link>
   <joint name="lidar_joint" type="fixed">
     <parent link="base_link" />
     <child link="sllidar_base_link"/>
-    <origin xyz="0 0 ${wheel_diameter / 2 + 0.1}"/>
+    <origin xyz="0 ${wheelbase_length / 2 - LiDAR_radius} ${wheel_diameter / 2 + 0.1}"/>
   </joint>
   <gazebo reference="sllidar_base_link">

Commit message: smart car spawned in met lidar

File: src/smart_car/urdf/smartcar.urdf (robot description, URDF)
Before this commit: robot smartcar, 8 links, 7 joints
Links:
- link back_left_wheel: geometry collision cylinder length=0.025 radius=0.032; visual cylinder length=0.025 radius=0.032
- link back_right_wheel: geometry collision cylinder length=0.025 radius=0.032; visual cylinder length=0.025 radius=0.032
- link front_left_wheel: geometry collision cylinder length=0.025 radius=0.032; visual cylinder length=0.025 radius=0.032
- link front_right_wheel: geometry collision cylinder length=0.025 radius=0.032; visual cylinder length=0.025 radius=0.032

File: src/smart_car/urdf/smartcar.urdf.xacro (robot description, xacro)
@@ -19,4 +19,10 @@
         </geometry>
       </visual>
+      <collision>
+        <origin xyz="0 0 0" rpy="0 0 0"/>
+        <geometry>
+          <cylinder radius="${wheel_diameter/2}" length="${wheel_width}"/>
+        </geometry>
+      </collision>
     </link>
     <joint name="${prefix}_wheel_joint" type="continuous">
@@ -33,5 +39,5 @@
       <mass value="1.0"/>
       <inertia ixx="0.01" ixy="0.0" ixz="0.0" iyy="0.01" iyz="0.0" izz="0.02"/>
-      <origin xyz="0 0 0"/>
+      <origin xyz="0 0 1"/>
     </inertial>
     <visual>
@@ -112,5 +118,6 @@
   </joint>
   <gazebo reference="sllidar_base_link">
-    <sensor type="ray" name="lidar_sensor">
+    <!-- <sensor type="ray" name="lidar_sensor">
+      <visualize>true</visualize>
       <update_rate>30.0</update_rate>
       <plugin name="gazebo_ros_ray_sensor" filename="libgazebo_ros_ray_sensor.so">
@@ -118,5 +125,30 @@
         <frameName>sllidar_base_link</frameName>
       </plugin>
-    </sensor>
+    </sensor> -->
+    <sensor name="lidar" type="ray">
+      <pose> 0 0 0 0 0 0 </pose>
+      <visualize>true</visualize>
+      <update_rate>10</update_rate>
+      <ray>
+          <scan>
+              <horizontal>
+                  <samples>360</samples>
+                  <min_angle>-3.14</min_angle>
+                  <max_angle>3.14</max_angle>
+              </horizontal>
+          </scan>
+          <range>
+              <min>0.3</min>
+              <max>12</max>
+          </range>
+      </ray>
+      <plugin name="lidar_plugin" filename="libgazebo_ros_ray_sensor.so">
+          <ros>
+              <argument>~/out:=scan</argument>
+          </ros>
+          <output_type>sensor_msgs/LaserScan</output_type>
+          <frame_name>sllidar_base_link</frame_name>
+      </plugin>
+  </sensor>
   </gazebo>
 </robot>
