Commit message: test

File: install/smart_car/share/smart_car/urdf/smartcar.urdf (robot description, URDF)
Before this commit: robot smartcar, 5 links, 4 joints
Links:
- added link chassis_link; visual box size=0.17 0.257 0.01
- link base_link: geometry 
Joints:
- added joint chassis_joint: type fixed, parent base_link, child chassis_link, origin xyz=0 0 0.032
- joint front_left_wheel_joint: origin xyz=0.085 -0.1285 0.032 rpy=0 1.5707963267948966 0 -> xyz=0.11000000000000001 -0.1285 0.032 rpy=0 1.5707963267948966 0
- joint front_right_wheel_joint: origin xyz=-0.085 -0.1285 0.032 rpy=0 1.5707963267948966 0 -> xyz=-0.11000000000000001 -0.1285 0.032 rpy=0 1.5707963267948966 0
- joint rear_left_wheel_joint: origin xyz=0.085 0.1285 0.032 rpy=0 1.5707963267948966 0 -> xyz=0.11000000000000001 0.1285 0.032 rpy=0 1.5707963267948966 0
- joint rear_right_wheel_joint: origin xyz=-0.085 0.1285 0.032 rpy=0 1.5707963267948966 0 -> xyz=-0.11000000000000001 0.1285 0.032 rpy=0 1.5707963267948966 0

File: install/smart_car/share/smart_car/urdf/smartcar.urdf.xacro (robot description, xacro)
@@ -22,12 +22,24 @@
     <visual>
       <geometry>
-        <box size="${wheelbase_width} ${wheelbase_length}  0.01"/>
-        <origin xyz="0 0 ${wheel_diameter / 2}"/>
+        <!-- <box size="${wheelbase_width} ${wheelbase_length}  0.01"/>
+        <origin xyz="0 0 ${wheel_diameter / 2}"/> -->
       </geometry>
     </visual>
   </link>
-  <xacro:wheel prefix="front_left"  parent="base_link" x="${wheelbase_width / 2}" y="-${wheelbase_length / 2}" z="${wheel_diameter / 2}"/>
-  <xacro:wheel prefix="front_right" parent="base_link" x="-${wheelbase_width / 2}" y="-${wheelbase_length / 2}" z="${wheel_diameter / 2}"/>
-  <xacro:wheel prefix="rear_left"   parent="base_link" x="${wheelbase_width / 2}" y="${wheelbase_length / 2}" z="${wheel_diameter / 2}"/>
-  <xacro:wheel prefix="rear_right"  parent="base_link" x="-${wheelbase_width / 2}" y="${wheelbase_length / 2}" z="${wheel_diameter / 2}"/>
+    <link name="chassis_link">
+    <visual>
+      <geometry>
+        <box size="${wheelbase_width} ${wheelbase_length}  0.01"/>
+      </geometry>
+    </visual>
+  </link>
+      <joint name="chassis_joint" type="fixed">
+      <parent link="base_link" />
+      <child link="chassis_link"/>
+      <origin xyz="0 0 ${wheel_diameter / 2}"/>
+  </joint>
+  <xacro:wheel prefix="front_left"  parent="base_link" x="${wheelbase_width / 2 + wheel_width}" y="-${wheelbase_length / 2}" z="${wheel_diameter / 2}"/>
+  <xacro:wheel prefix="front_right" parent="base_link" x="-${wheelbase_width / 2 + wheel_width}" y="-${wheelbase_length / 2}" z="${wheel_diameter / 2}"/>
+  <xacro:wheel prefix="rear_left"   parent="base_link" x="${wheelbase_width / 2 + wheel_width}" y="${wheelbase_length / 2}" z="${wheel_diameter / 2}"/>
+  <xacro:wheel prefix="rear_right"  parent="base_link" x="-${wheelbase_width / 2 + wheel_width}" y="${wheelbase_length / 2}" z="${wheel_diameter / 2}"/>
 </robot>

File: src/smart_car/urdf/smartcar.urdf.xacro (robot description, xacro)
@@ -31,11 +31,15 @@
       <geometry>
         <box size="${wheelbase_width} ${wheelbase_length}  0.01"/>
-        <origin xyz="0 0 ${wheel_diameter / 2}"/>
       </geometry>
     </visual>
   </link>
-  <xacro:wheel prefix="front_left"  parent="base_link" x="${wheelbase_width / 2}" y="-${wheelbase_length / 2}" z="${wheel_diameter / 2}"/>
-  <xacro:wheel prefix="front_right" parent="base_link" x="-${wheelbase_width / 2}" y="-${wheelbase_length / 2}" z="${wheel_diameter / 2}"/>
-  <xacro:wheel prefix="rear_left"   parent="base_link" x="${wheelbase_width / 2}" y="${wheelbase_length / 2}" z="${wheel_diameter / 2}"/>
-  <xacro:wheel prefix="rear_right"  parent="base_link" x="-${wheelbase_width / 2}" y="${wheelbase_length / 2}" z="${wheel_diameter / 2}"/>
+      <joint name="chassis_joint" type="fixed">
+      <parent link="base_link" />
+      <child link="chassis_link"/>
+      <origin xyz="0 0 ${wheel_diameter / 2}"/>
+  </joint>
+  <xacro:wheel prefix="front_left"  parent="base_link" x="${wheelbase_width / 2 + wheel_width}" y="-${wheelbase_length / 2}" z="${wheel_diameter / 2}"/>
+  <xacro:wheel prefix="front_right" parent="base_link" x="-${wheelbase_width / 2 + wheel_width}" y="-${wheelbase_length / 2}" z="${wheel_diameter / 2}"/>
+  <xacro:wheel prefix="back_left"   parent="base_link" x="${wheelbase_width / 2 + wheel_width}" y="${wheelbase_length / 2}" z="${wheel_diameter / 2}"/>
+  <xacro:wheel prefix="back_right"  parent="base_link" x="-${wheelbase_width / 2 + wheel_width}" y="${wheelbase_length / 2}" z="${wheel_diameter / 2}"/>
 </robot>

Commit message: car gazebo plugin issue

File: install/smart_car/share/smart_car/urdf/smartcar.urdf (robot description, URDF)
Before this commit: robot smartcar, 6 links, 5 joints
Links:
- removed link rear_left_wheel
- removed link rear_right_wheel
- added link back_left_wheel, mass 0.2; collision cylinder length=0.025 radius=0.032; visual cylinder length=0.025 radius=0.032
- added link back_right_wheel, mass 0.2; collision cylinder length=0.025 radius=0.032; visual cylinder length=0.025 radius=0.032
- added link imu_link, mass 0.05; collision box size=0.1 0.1 0.1; visual box size=0.05 0.05 0.05
- added link sllidar_base_link, mass 0.05; collision cylinder length=0.1 radius=0.03; visual cylinder length=0.1 radius=0.03
- link chassis_link: mass None -> 1.0
- link front_left_wheel: mass None -> 0.2; geometry collision cylinder length=0.025 radius=0.032; visual cylinder length=0.025 radius=0.032
- link front_right_wheel: mass None -> 0.2; geometry collision cylinder length=0.025 radius=0.032; visual cylinder length=0.025 radius=0.032
Joints:
- removed joint rear_left_wheel_joint
- removed joint rear_right_wheel_joint
- added joint back_left_wheel_joint: type continuous, parent base_link, child back_left_wheel, origin xyz=0.11000000000000001 0.1285 0.032 rpy=0 1.5707963267948966 0
- added joint back_right_wheel_joint: type continuous, parent base_link, child back_right_wheel, origin xyz=-0.11000000000000001 0.1285 0.032 rpy=0 1.5707963267948966 0
- added joint imu_joint: type fixed, parent base_link, child imu_link, origin xyz=0 0 0.082
- added joint lidar_joint: type fixed, parent base_link, child sllidar_base_link, origin xyz=0 0.0985 0.132

File: install/smart_car/share/smart_car/urdf/smartcar.urdf.xacro (robot description, xacro)
@@ -1,10 +1,17 @@
 <?xml version="1.0"?>
 <robot xmlns:xacro="http://www.ros.org/wiki/xacro" name="smartcar">
+  <!--Xacro properties and macros-->
   <xacro:property name="wheel_diameter" value="0.064" />
   <xacro:property name="wheel_width" value="0.025" />
   <xacro:property name="wheelbase_length" value="0.257" />
   <xacro:property name="wheelbase_width" value="0.17" />
+  <xacro:property name="LiDAR_radius" value="0.03" />
   <xacro:macro name="wheel" params="prefix parent x y z">
     <link name="${prefix}_wheel">
+      <inertial>
+        <mass value="0.2"/>
+        <inertia ixx="0.0001" ixy="0.0" ixz="0.0" iyy="0.0001" iyz="0.0" izz="0.0002"/>
+        <origin xyz="0 0 0"/>
+      </inertial>
       <visual>
         <geometry>
@@ -12,20 +19,26 @@
         </geometry>
       </visual>
+      <collision>
+        <origin xyz="0 0 0" rpy="0 0 0"/>
+        <geometry>
+          <cylinder radius="${wheel_diameter/2}" length="${wheel_width}"/>
+        </geometry>
+      </collision>
     </link>
     <joint name="${prefix}_wheel_joint" type="continuous">
       <parent link="${parent}" />
       <child link="${prefix}_wheel"/>
-       <origin xyz="${x} ${y} ${z}" rpy="0 ${pi/2} 0"/>
+      <origin xyz="${x} ${y} ${z}" rpy="0 ${pi/2} 0"/>
     </joint>
   </xacro:macro>
+  <!--Body-->
   <link name="base_link">
-    <visual>
-      <geometry>
-        <!-- <box size="${wheelbase_width} ${wheelbase_length}  0.01"/>
-        <origin xyz="0 0 ${wheel_diameter / 2}"/> -->
-      </geometry>
-    </visual>
   </link>
-    <link name="chassis_link">
+  <link name="chassis_link">
+    <inertial>
+      <mass value="1.0"/>
+      <inertia ixx="0.01" ixy="0.0" ixz="0.0" iyy="0.01" iyz="0.0" izz="0.02"/>
+      <origin xyz="0 0 1"/>
+    </inertial>
     <visual>
       <geometry>
@@ -34,12 +47,103 @@
     </visual>
   </link>
-      <joint name="chassis_joint" type="fixed">
-      <parent link="base_link" />
-      <child link="chassis_link"/>
-      <origin xyz="0 0 ${wheel_diameter / 2}"/>
+  <joint name="chassis_joint" type="fixed">
+    <parent link="base_link" />
+    <child link="chassis_link"/>
+    <origin xyz="0 0 ${wheel_diameter / 2}"/>
   </joint>
-  <xacro:wheel prefix="front_left"  parent="base_link" x="${wheelbase_width / 2 + wheel_width}" y="-${wheelbase_length / 2}" z="${wheel_diameter / 2}"/>
+  <xacro:wheel prefix="front_left" parent="base_link" x="${wheelbase_width / 2 + wheel_width}" y="-${wheelbase_length / 2}" z="${wheel_diameter / 2}"/>
   <xacro:wheel prefix="front_right" parent="base_link" x="-${wheelbase_width / 2 + wheel_width}" y="-${wheelbase_length / 2}" z="${wheel_diameter / 2}"/>
-  <xacro:wheel prefix="rear_left"   parent="base_link" x="${wheelbase_width / 2 + wheel_width}" y="${wheelbase_length / 2}" z="${wheel_diameter / 2}"/>
-  <xacro:wheel prefix="rear_right"  parent="base_link" x="-${wheelbase_width / 2 + wheel_width}" y="${wheelbase_length / 2}" z="${wheel_diameter / 2}"/>
+  <xacro:wheel prefix="back_left" parent="base_link" x="${wheelbase_width / 2 + wheel_width}" y="${wheelbase_length / 2}" z="${wheel_diameter / 2}"/>
+  <xacro:wheel prefix="back_right" parent="base_link" x="-${wheelbase_width / 2 + wheel_width}" y="${wheelbase_length / 2}" z="${wheel_diameter / 2}"/>
+  <!--Sensors-->
+  <!--IMU-->
+  <link name="imu_link">
+    <visual>
+      <geometry>
+        <box size="0.05 0.05 0.05"/>
+      </geometry>
+    </visual>
+    <collision>
+      <origin xyz="0 0 0" rpy="0 0 0"/>
+      <geometry>
+          <box size="0.1 0.1 0.1"/>
+      </geometry>
+    </collision>
+    <inertial>
+      <mass value="0.05"/>
+      <inertia ixx="0.01" ixy="0.0" ixz="0.0" iyy="0.01" iyz="0.0" izz="0.02"/>
+      <origin xyz="0 0 0"/>
+    </inertial>
+  </link>
+  <joint name="imu_joint" type="fixed">
+    <parent link="base_link" />
+    <child link="imu_link"/>
+    <origin xyz="0 0 ${wheel_diameter / 2 + 0.05}"/>
+  </joint>
+  <gazebo reference="imu_link">
+    <sensor type="imu" name="imu_sensor">
+      <always_on>true</always_on>
+      <update_rate>30.0</update_rate>
+      <plugin name="gazebo_ros_imu" filename="libgazebo_ros_imu.so">
+        <ros>
+          <namespace>/imu</namespace>
+          <remapping>~/out:=/imu/data</remapping>
+        </ros>
+      </plugin>
+    </sensor>
+  </gazebo>
+  <!-- LiDAR -->
+  <link name="sllidar_base_link">
+    <visual>
+      <geometry>
+        <cylinder radius="${LiDAR_radius}" length="0.1"/>
+      </geometry>
+    </visual>
+    <collision>
+      <origin xyz="0 0 0" rpy="0 0 0"/>
+      <geometry>
+        <cylinder radius="${LiDAR_radius}" length="0.1"/>
+      </geometry>
+    </collision>
+    <inertial>
+      <mass value="0.05"/>
+      <inertia ixx="0.01" ixy="0.0" ixz="0.0" iyy="0.01" iyz="0.0" izz="0.02"/>
+      <origin xyz="0 0 0"/>
+    </inertial>
+  </link>
+  <joint name="lidar_joint" type="fixed">
+    <parent link="base_link" />
+    <child link="sllidar_base_link"/>
+    <origin xyz="0 ${wheelbase_length / 2 - LiDAR_radius} ${wheel_diameter / 2 + 0.1}"/>
+  </joint>
+  <gazebo reference="sllidar_base_link">
+    <sensor name="lidar" type="ray">
+      <pose> 0 0 0 0 0 0 </pose>
+      <visualize>true</visualize>
+      <update_rate>10</update_rate>
+      <ray>
+          <scan>
+              <horizontal>
+                  <samples>360</samples>
+                  <min_angle>-${pi}</min_angle>
+                  <max_angle>${pi}</max_angle>
+              </horizontal>
+          </scan>
+          <range>
+              <min>0.3</min>
+              <max>12</max>
+          </range>
+      </ray>
+      <plugin name="lidar_plugin" filename="libgazebo_ros_ray_sensor.so">
+          <ros>
+              <argument>~/out:=scan</argument>
+          </ros>
+          <output_type>sensor_msgs/LaserScan</output_type>
+          <frame_name>sllidar_base_link</frame_name>
+      </plugin>
+  </sensor>
+  </gazebo>
+  <gazebo>
+    <plugin name="car_gazebo_plugin" filename="libcar_gazebo_plugin.so"></plugin>
+  </gazebo>
 </robot>

File: src/smart_car/urdf/smartcar.urdf.xacro (robot description, xacro)
@@ -118,12 +118,4 @@
   </joint>
   <gazebo reference="sllidar_base_link">
-    <!-- <sensor type="ray" name="lidar_sensor">
-      <visualize>true</visualize>
-      <update_rate>30.0</update_rate>
-      <plugin name="gazebo_ros_ray_sensor" filename="libgazebo_ros_ray_sensor.so">
-        <topic>/scan</topic>
-        <frameName>sllidar_base_link</frameName>
-      </plugin>
-    </sensor> -->
     <sensor name="lidar" type="ray">
       <pose> 0 0 0 0 0 0 </pose>
@@ -134,6 +126,6 @@
               <horizontal>
                   <samples>360</samples>
-                  <min_angle>-3.14</min_angle>
-                  <max_angle>3.14</max_angle>
+                  <min_angle>-${pi}</min_angle>
+                  <max_angle>${pi}</max_angle>
               </horizontal>
           </scan>
@@ -152,3 +144,6 @@
   </sensor>
   </gazebo>
+  <gazebo>
+    <plugin name="car_gazebo_plugin" filename="libcar_gazebo_plugin.so"></plugin>
+  </gazebo>
 </robot>
