Commit message: i am the smartest man alive. nav2 works

File: src/smartcar_simulation/urdf/smartcar.urdf (robot description, URDF)
Before this commit: robot smartcar, 10 links, 9 joints
Links:
- added link base_footprint, mass 1; visual box size=0.257 0.17 0.01
Joints:
- added joint base_footprint_joint: type fixed, parent base_link, child base_footprint

File: src/smartcar_simulation/urdf/smartcar.urdf.xacro (robot description, xacro)
@@ -91,4 +91,20 @@
   <link name="base_link">
   </link>
+  <link name="base_footprint">
+    <inertial>
+      <mass value="1"/>
+      <inertia ixx="0.01" ixy="0.0" ixz="0.0" iyy="0.01" iyz="0.0" izz="0.02"/>
+      <origin xyz="0 0 0"/>
+    </inertial>
+    <visual>
+      <geometry>
+        <box size="${wheelbase_length} ${wheelbase_width} 0.01"/>
+      </geometry>
+    </visual>
+  </link>
+  <joint name="base_footprint_joint" type="fixed">
+    <parent link="base_link" />
+    <child link="base_footprint"/>
+  </joint>
   <link name="chassis_link">
     <inertial>
